Commit message: Add robot model visualization and laser frame

File: week06/ros2_ws/src/robot_motion_sim/urdf/robot.urdf (robot description, URDF)
Before this commit: robot simple_diff_drive_robot, 4 links, 3 joints
Links:
- added link laser_link; visual box size=0.06 0.04 0.03
Joints:
- added joint laser_joint: type fixed, parent base_link, child laser_link, origin xyz=0.18 0 0.14 rpy=0 0 0
