Commit message: Connect AMR control to Gazebo Sim

File: week09/amr_ws/src/amr_description/urdf/amr_base.xacro (robot description, xacro)
@@ -11,4 +11,5 @@
   <xacro:property name="wheel_separation" value="0.36"/>
   <xacro:property name="caster_radius" value="0.035"/>
+  <xacro:property name="base_clearance" value="0.02"/>
   <!-- Approximate masses -->
   <xacro:property name="base_mass" value="8.0"/>
@@ -31,6 +32,6 @@
     </inertial>
   </xacro:macro>
-  <xacro:macro name="cylinder_inertia_z" params="mass radius length">
-    <!-- Cylinder aligned with z-axis -->
+  <xacro:macro name="cylinder_inertia_y" params="mass radius length">
+    <!-- Cylinder aligned with y-axis -->
     <inertial>
       <mass value="${mass}"/>
@@ -40,7 +41,7 @@
         ixy="0.0"
         ixz="0.0"
-        iyy="${(mass/12.0) * (3*radius*radius + length*length)}"
+        iyy="${0.5 * mass * radius * radius}"
         iyz="0.0"
-        izz="${0.5 * mass * radius * radius}"/>
+        izz="${(mass/12.0) * (3*radius*radius + length*length)}"/>
     </inertial>
   </xacro:macro>
@@ -63,5 +64,7 @@
   <link name="base_link">
     <visual>
-      <origin xyz="0 0 ${base_height/2.0}" rpy="0 0 0"/>
+      <origin
+        xyz="0 0 ${wheel_radius + base_clearance + base_height/2.0}"
+        rpy="0 0 0"/>
       <geometry>
         <box size="${base_length} ${base_width} ${base_height}"/>
@@ -70,5 +73,7 @@
     </visual>
     <collision>
-      <origin xyz="0 0 ${base_height/2.0}" rpy="0 0 0"/>
+      <origin
+        xyz="0 0 ${wheel_radius + base_clearance + base_height/2.0}"
+        rpy="0 0 0"/>
       <geometry>
         <box size="${base_length} ${base_width} ${base_height}"/>
@@ -99,5 +104,5 @@
       </geometry>
     </collision>
-    <xacro:cylinder_inertia_z
+    <xacro:cylinder_inertia_y
       mass="${wheel_mass}"
       radius="${wheel_radius}"
@@ -127,5 +132,5 @@
       </geometry>
     </collision>
-    <xacro:cylinder_inertia_z
+    <xacro:cylinder_inertia_y
       mass="${wheel_mass}"
       radius="${wheel_radius}"
@@ -186,3 +191,14 @@
     <origin xyz="${-base_length/2.0 + 0.08} 0 ${caster_radius}" rpy="0 0 0"/>
   </joint>
+  <!-- ========================= -->
+  <!-- Gazebo friction settings  -->
+  <!-- ========================= -->
+  <gazebo reference="left_wheel_link">
+    <mu1>1.0</mu1>
+    <mu2>1.0</mu2>
+  </gazebo>
+  <gazebo reference="right_wheel_link">
+    <mu1>1.0</mu1>
+    <mu2>1.0</mu2>
+  </gazebo>
 </robot>

Commit message: Add Gazebo GPU LiDAR simulation

File: week09/amr_ws/src/amr_description/urdf/amr_base.xacro (robot description, xacro)
@@ -12,4 +12,8 @@
   <xacro:property name="caster_radius" value="0.035"/>
   <xacro:property name="base_clearance" value="0.02"/>
+  <xacro:property name="lidar_radius" value="0.05"/>
+  <xacro:property name="lidar_height" value="0.06"/>
+  <xacro:property name="lidar_mass" value="0.3"/>
+  <xacro:property name="lidar_z" value="${wheel_radius + base_clearance + base_height + lidar_height/2.0}"/>
   <!-- Approximate masses -->
   <xacro:property name="base_mass" value="8.0"/>
@@ -190,4 +194,36 @@
     <child link="back_caster_link"/>
     <origin xyz="${-base_length/2.0 + 0.08} 0 ${caster_radius}" rpy="0 0 0"/>
+  </joint>
+  <!-- ========================= -->
+  <!-- LiDAR                     -->
+  <!-- ========================= -->
+  <link name="lidar_link">
+    <visual>
+      <origin xyz="0 0 0" rpy="0 0 0"/>
+      <geometry>
+        <cylinder radius="${lidar_radius}" length="${lidar_height}"/>
+      </geometry>
+      <material name="black"/>
+    </visual>
+    <collision>
+      <origin xyz="0 0 0" rpy="0 0 0"/>
+      <geometry>
+        <cylinder radius="${lidar_radius}" length="${lidar_height}"/>
+      </geometry>
+    </collision>
+    <inertial>
+      <mass value="${lidar_mass}"/>
+      <origin xyz="0 0 0" rpy="0 0 0"/>
+      <inertia
+        ixx="${(1.0/12.0) * lidar_mass * (3.0 * lidar_radius * lidar_radius + lidar_height * lidar_height)}"
+        iyy="${(1.0/12.0) * lidar_mass * (3.0 * lidar_radius * lidar_radius + lidar_height * lidar_height)}"
+        izz="${0.5 * lidar_mass * lidar_radius * lidar_radius}"
+        ixy="0.0" ixz="0.0" iyz="0.0"/>
+    </inertial>
+  </link>
+  <joint name="lidar_joint" type="fixed">
+    <parent link="base_link"/>
+    <child link="lidar_link"/>
+    <origin xyz="0 0 ${lidar_z}" rpy="0 0 0"/>
   </joint>
   <!-- ========================= -->
@@ -202,3 +238,27 @@
     <mu2>1.0</mu2>
   </gazebo>
+  <gazebo reference="lidar_link">
+    <sensor name="lidar_sensor" type="gpu_lidar">
+      <update_rate>10</update_rate>
+      <topic>scan</topic>
+      <gz_frame_id>lidar_link</gz_frame_id>
+      <lidar>
+        <scan>
+          <horizontal>
+            <samples>720</samples>
+            <resolution>1</resolution>
+            <min_angle>-3.14159</min_angle>
+            <max_angle>3.14159</max_angle>
+          </horizontal>
+        </scan>
+        <range>
+          <min>0.12</min>
+          <max>12.0</max>
+          <resolution>0.01</resolution>
+        </range>
+      </lidar>
+      <always_on>true</always_on>
+      <visualize>true</visualize>
+    </sensor>
+  </gazebo>
 </robot>
